Commit message: Change initial pose and file structure
Change robot initial pose to 'pickup' pose, and modified '.xml' files structure using <mujocoinclude> tag.

File: e05/urdf/e05.urdf (robot description, URDF)
Before this commit: robot e05, 8 links, 7 joints
Joints:
- joint joint1: origin xyz=0 0 0.0735 rpy=0 0 0 -> xyz=0 0 0.0735 rpy=0 0 1.5707963267949
- joint joint3: origin xyz=0 -0.38 0 rpy=0 0 1.57079632679489 -> xyz=0 -0.38 0 rpy=0 0 0
- joint joint5: origin xyz=0 0 -0.42 rpy=-1.5708 0 0 -> xyz=0 0 -0.42 rpy=-1.5708 1.5708 0
